File: hardware/ESC.kicad_sch (KiCad schematic)
At the start: 36 parts, among them Q1 SP40N01GHNK, Q11 SP40N01GHNK, Q16 SP40N01GHNK, Q2 SP40N01GHNK, Q21 SP40N01GHNK, Q6 SP40N01GHNK, U2 AT32F421G8U7, U4 NSG2065Q

Commit message: schematics: fill Manufacturer on every part with an LCSC number
Every placed part now carries LCSC + Manufacturer + MPN, manufacturer names
from the LCSC catalogue. Feeds OpenDrone-Scripts kicad/universal_bom.py for
quoting outside JLCPCB; its output matches the rev3.2 Toolkit BOM exactly
(21 lines, 213 placements).

kicad-skip reflowed the files on write; S-expression structural diff against
the originals shows only the property changes, ERC identical before and
after (350 violations, same categories).

Co-Authored-By: Claude Fable 5 <noreply@anthropic.com>
Parts:
- C32, C36, C53: Manufacturer (none) -> Samsung Electro-Mechanics
- C48, C49, C50, C57: Manufacturer (none) -> muRata
- Q1, Q11, Q16, Q2, Q21, Q6: Manufacturer (none) -> Siliup
- R18, R19, R20, R25, R27, R28, R30, R31, R33, R84: Manufacturer (none) -> YAGEO
- R23, R26, R29, R32, R42, R55, R62, R76, R80: Manufacturer (none) -> UNI-ROYAL
- U4: Manufacturer (none) -> WXNSIC
