File: hardware/4in1-panel.kicad_pcb (KiCad board)
At the start: 6 copper layers, 41.6 x 42.5 mm, 404 parts, among them J1 SM08B-SRSS-TB, Q1 C22385416, Q1 DOY180N03T, Q10 C22385416, Q10 DOY180N03T, Q11 C22385416, Q11 DOY180N03T, Q12 C22385416, Q12 DOY180N03T, Q13 C22385416, Q13 DOY180N03T, Q14 C22385416, Q14 DOY180N03T, Q15 C22385416, Q15 DOY180N03T, Q16 C22385416, Q16 DOY180N03T, Q17 C22385416, Q17 DOY180N03T, Q18 C22385416, Q18 DOY180N03T, Q19 C22385416, Q19 DOY180N03T, Q2 C22385416, Q2 DOY180N03T, Q20 C22385416, Q20 DOY180N03T, Q21 C22385416, Q21 DOY180N03T, Q22 C22385416, Q22 DOY180N03T, Q23 C22385416, Q23 DOY180N03T, Q24 C22385416, Q24 DOY180N03T, Q3 C22385416, Q3 DOY180N03T, Q4 C22385416, Q4 DOY180N03T, Q5 C22385416, Q5 DOY180N03T, Q6 C22385416, Q6 DOY180N03T, Q7 C22385416, Q7 DOY180N03T, Q8 C22385416, Q8 DOY180N03T, Q9 C22385416, Q9 DOY180N03T, U1 TLV76733DRVR, U10 AT32F421G8U7, U10 NSG2065Q, U11 NSG2065Q, U12 INA186A3IDCKR, U13 LMR54406DBVR, U14 FTC160808S4R7MBCA, U15 TLV76733DRVR, U2 AT32F421G8U7, U3 NSG2065Q, U4 NSG2065Q, U5 AT32F421G8U7, U5 FTC160808S4R7MBCA, U6 AT32F421G8U7, U6 NSG2065Q, U7 AT32F421G8U7, U7 NSG2065Q, U8 AT32F421G8U7, U8 NSG2065Q, U9 AT32F421G8U7, U9 NSG2065Q

Commit message: Swap bulk caps to FH 1206B475K500NT 4.7uF 50V (C29823)
Replaces Samsung CL31B106KBHNNNE 10uF (C89632) on schematic symbols
C2/C3/C6 and all 70 panel-board footprints. Cost cut: NextPCB priced
the 10uF at $0.218/pc; the FH part is ~$0.03 and a JLCPCB basic part.
Single-board file 4in1.kicad_pcb also swapped (52 footprints) but left
uncommitted: it carries unrelated WIP silkscreen changes.

Co-Authored-By: Claude Fable 5 <noreply@anthropic.com>
Parts:
- C100, C101, C105, C106, C107, C108, C13, C14, C15, C16, C17, C18, C19, C2, C20, C24, C25, C26, C27, C28, C29, C3, C30, C31, C43, C44, C45, C6 (x3), C69, C7, C70, C71, C72, C79, C8, C80, C82, C83, C84, C85, C87, C88, C9, C95, C96, C97, C98, C99, CL32, CL33, CL34, CL35, CL36, CL38, CL39, CL40, CL42, CL43, CL44, CL45, CL46, CL47, CL48, CL49, CL50, CL51, CL54, CL55: value 10uF -> 4.7uF
