File: hardware/4in1.kicad_pcb (KiCad board)
At the start: 6 copper layers, 41.6 x 42.5 mm, 222 parts, among them J1 SM08B-SRSS-TB, Q1 SP40N01GHNK, Q10 SP40N01GHNK, Q11 SP40N01GHNK, Q12 SP40N01GHNK, Q13 SP40N01GHNK, Q14 SP40N01GHNK, Q15 SP40N01GHNK, Q16 SP40N01GHNK, Q17 SP40N01GHNK, Q18 SP40N01GHNK, Q19 SP40N01GHNK, Q2 SP40N01GHNK, Q20 SP40N01GHNK, Q21 SP40N01GHNK, Q22 SP40N01GHNK, Q23 SP40N01GHNK, Q24 SP40N01GHNK, Q3 SP40N01GHNK, Q4 SP40N01GHNK, Q5 SP40N01GHNK, Q6 SP40N01GHNK, Q7 SP40N01GHNK, Q8 SP40N01GHNK, Q9 SP40N01GHNK, U10 NSG2065Q, U12 INA186A3IDCKR, U13 LMR54406DBVR, U14 FTC160808S4R7MBCA, U15 TLV76733DRVR, U2 AT32F421G8U7, U4 NSG2065Q, U5 AT32F421G8U7, U6 NSG2065Q, U7 AT32F421G8U7, U8 NSG2065Q, U9 AT32F421G8U7

Commit message: AGENTS: record rev3.3; rev silk synced by pipeline
Co-Authored-By: Claude Fable 5 <noreply@anthropic.com>
Other:
- board text added: "REV3.3"
- board text removed: "REV3.2"
Changed lines of the file:
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@@
 	(paper "A4")
 	(title_block
-		(rev "rev3.2")
+		(rev "rev3.3")
 	)
 	(layers
@@
 		)
 	)
-	(gr_text "REV3.2"
+	(gr_text "REV3.3"
 		(at 87.12 56.53 0)
 		(layer "B.SilkS")
@@
 			(justify left bottom mirror)
 		)
-		(render_cache "REV3.2" 0
+		(render_cache "REV3.3" 0
 			(polygon
 				(pts
@@
 			(polygon
 				(pts
-					(xy 83.059511 56.224) (xy 83.059511 55.441116) (xy 83.051258 55.374893) (xy 83.027065 55.316478)
-					(xy 82.986092 55.263832) (xy 82.933388 55.222921) (xy 82.874205 55.198631) (xy 82.80639 55.190303)
-					(xy 82.616357 55.190303) (xy 82.616357 54.753523) (xy 82.764624 54.753523) (xy 82.764624 55.043024)
-					(xy 83.059511 55.043024) (xy 83.059511 54.70934) (xy 83.051224 54.642106) (xy 83.027049 54.583432)
-					(xy 82.986311 54.531177) (xy 82.933733 54.490723) (xy 82.87462 54.46667) (xy 82.80683 54.458417)
-					(xy 82.574262 54.458417) (xy 82.50812 54.466599) (xy 82.449388 54.490636) (xy 82.396099 54.531397)
-					(xy 82.354516 54.583896) (xy 82.329898 54.642746) (xy 82.32147 54.710109) (xy 82.32147 55.236245)
-					(xy 82.329839 55.301929) (xy 82.354422 55.359974) (xy 82.396209 55.412429) (xy 82.44957 55.453182)
-					(xy 82.508411 55.477224) (xy 82.574701 55.485409) (xy 82.764624 55.485409) (xy 82.764624 55.928893)
-					(xy 82.616357 55.928893) (xy 82.616357 55.634886) (xy 82.32147 55.634886) (xy 82.32147 56.224)
+					(xy 82.813754 56.224) (xy 82.881507 56.215693) (xy 82.940618 56.191472) (xy 82.993236 56.15069)
+					(xy 83.034012 56.09807) (xy 83.058236 56.038925) (xy 83.066545 55.971098) (xy 83.066545 55.634886)
+					(xy 82.771659 55.634886) (xy 82.771659 55.928893) (xy 82.623391 55.928893) (xy 82.623391 55.604551)
+					(xy 82.631909 55.559705) (xy 82.657683 55.52091) (xy 82.695924 55.494345) (xy 82.742643 55.485409)
+					(xy 82.920366 55.485409) (xy 82.920366 55.190303) (xy 82.742643 55.190303) (xy 82.695872 55.181512)
+					(xy 82.657683 55.155461) (xy 82.631896 55.117215) (xy 82.623391 55.07303) (xy 82.623391 54.753523)
+					(xy 82.771659 54.753523) (xy 82.771659 55.043024) (xy 83.066545 55.043024) (xy 83.066545 54.70934)
+					(xy 83.058248 54.642114) (xy 83.034039 54.58344) (xy 82.993236 54.531177) (xy 82.940657 54.490723)
+					(xy 82.881544 54.46667) (xy 82.813754 54.458417) (xy 82.581296 54.458417) (xy 82.515147 54.466588)
+					(xy 82.456415 54.490592) (xy 82.403133 54.531287) (xy 82.361542 54.583714) (xy 82.336928 54.642456)
+					(xy 82.328504 54.709669) (xy 82.328504 55.086658) (xy 82.337022 55.153805) (xy 82.361937 55.212543)
+					(xy 82.404122 55.265041) (xy 82.477212 55.337911) (xy 82.404122 55.41133) (xy 82.361966 55.464185)
+					(xy 82.337034 55.523395) (xy 82.328504 55.591142) (xy 82.328504 55.970769) (xy 82.33694 56.038582)
+					(xy 82.36157 56.097796) (xy 82.403133 56.15058) (xy 82.456453 56.191604) (xy 82.515183 56.215776)
+					(xy 82.581296 56.224)
 				)
 			)
