File: hardware/4in1.kicad_sch (KiCad schematic)
At the start: 29 parts, among them J1 SM08B-SRSS-TB, U12 INA186A3IDCKR, U13 LMR54406DBVR, U14 FTC160808S4R7MBCA, U15 TLV76733DRVR

Commit message: schematics: fill Manufacturer on every part with an LCSC number
Every placed part now carries LCSC + Manufacturer + MPN, manufacturer names
from the LCSC catalogue. Feeds OpenDrone-Scripts kicad/universal_bom.py for
quoting outside JLCPCB; its output matches the rev3.2 Toolkit BOM exactly
(21 lines, 213 placements).

kicad-skip reflowed the files on write; S-expression structural diff against
the originals shows only the property changes, ERC identical before and
after (350 violations, same categories).

Co-Authored-By: Claude Fable 5 <noreply@anthropic.com>
Parts:
- C2, C3, C4, C40, C41, C47, C51, C6, C86: Manufacturer (none) -> Samsung Electro-Mechanics
- C42, R121: Manufacturer (none) -> YAGEO
- C74, C75, C76, C81, C93, C94: Manufacturer (none) -> muRata
- J1: Manufacturer (none) -> JST
- R120: Manufacturer (none) -> RALEC
- R73, R89, R90: Manufacturer (none) -> UNI-ROYAL
- Rsense1, Rsense2: Manufacturer (none) -> Yezhan
- U14: Manufacturer (none) -> cjiang

Commit message: Swap bulk caps to FH 1206B475K500NT 4.7uF 50V (C29823)
Replaces Samsung CL31B106KBHNNNE 10uF (C89632) on schematic symbols
C2/C3/C6 and all 70 panel-board footprints. Cost cut: NextPCB priced
the 10uF at $0.218/pc; the FH part is ~$0.03 and a JLCPCB basic part.
Single-board file 4in1.kicad_pcb also swapped (52 footprints) but left
uncommitted: it carries unrelated WIP silkscreen changes.

Co-Authored-By: Claude Fable 5 <noreply@anthropic.com>
Parts:
- C2, C3, C6: value 10uF -> 4.7uF; Cost 0.05129 -> (none); LCSC C89632 -> C29823; MPN CL31B106KBHNNNE -> 1206B475K500NT; Manufacturer Samsung Electro-Mechanics -> FH

Commit message: Swap bulk caps to CCTC TCC1206X7R475K500HT (C380366)
FH C29823 was picked for its JLC-basic price; at LCSC retail it costs
USD 0.19/pc and we are no longer using JLCPCB assembly. CCTC part is
~USD 0.073/pc at 4k+ volume, same 4.7uF 10% 50V X7R 1206 class.
Fields only (LCSC/MPN/Manufacturer), no value, footprint or net changes.

Co-Authored-By: Claude Fable 5 <noreply@anthropic.com>
Parts:
- C2, C3, C6: LCSC C29823 -> C380366; MPN 1206B475K500NT -> TCC1206X7R475K500HT; Manufacturer FH -> CCTC
